File: Schem/Schem.kicad_sch (KiCad schematic)
At the start: 68 parts, among them IC1 MCP73831T-2ACI_OT, IC2 MCP1725-3302E_MC, IC3 MCP1725-3302E_MC, IC4 BQ25176MDSGR, J1 Conn_01x04, J2 Conn_01x02, J3 Conn_01x04, J4 Conn_01x02, Q1 BC547, Q2 BC547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

Commit message: updated todo
Parts:
- added R23: 33R, Resistor_SMD:R_0805_2012Metric_Pad1.20x1.40mm_HandSolder, symbol Device:R
Connections:
- net rst_to_shdn: now also R23.2; no longer 998-MIC2779L-2YM5TR1.4 (~RST_RST)
- new net: 998-MIC2779L-2YM5TR1.4 (~RST_RST), R23.1
Other:
- moved on the sheet: C12, C13, C14, C23, C24, D9

Commit message: added TODOs, calculated supervisor
Parts:
- added C16: 10 μF, Capacitor_THT:C_Rect_L16.5mm_W4.7mm_P15.00mm_MKT, symbol Device:C
- added C17: 0.1μF, Capacitor_THT:C_Rect_L16.5mm_W4.7mm_P15.00mm_MKT, symbol Device:C
- added C25: 1μF, Capacitor_THT:C_Rect_L16.5mm_W4.7mm_P15.00mm_MKT, symbol Device:C
- added J5____JTAG: Conn_01x04, symbol Connector_Generic:Conn_01x04
- added R24: 10KR, Resistor_SMD:R_0805_2012Metric_Pad1.20x1.40mm_HandSolder, symbol Device:R
- added R25, R26, R27, R28: 100R, Resistor_SMD:R_0805_2012Metric_Pad1.20x1.40mm_HandSolder, symbol Device:R
- R20: value 640KR -> 660kR
- R21: value 56KR -> 20KR
- R22: value 340kR -> 360kR
Connections:
- net +3V3: now also C16.2, C17.2, R24.1
- net GND: now also C16.1, C17.1, C25.1
- net at D8.2 (A): now also U2.30 (IO18); no longer U2.16 (IO13)
- net at U2.3 (EN): now also C25.2, R24.2
- new net: J5____JTAG.3 (Pin_3), R27.2
- new net: J5____JTAG.1 (Pin_1), R25.2
- new net: J5____JTAG.2 (Pin_2), R26.2
- new net: J5____JTAG.4 (Pin_4), R28.2
Other:
- moved on the sheet: 998-MIC2779L-2YM5TR1, C1, C10, C11, C12, C13, C14, C15, C18, C19, C2, C20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

Commit message: updated gitIgnore
Parts:
- added C26: 999 μF, Capacitor_THT:C_Rect_L16.5mm_W4.7mm_P15.00mm_MKT, symbol Device:C
Connections:
- net GND: now also C26.2
- net V_BAT_LOADER_IN: now also C26.1
Other:
- moved on the sheet: C12, C13, C14, C23, C24, D6, D8, D9, J3, R12

Commit message: minor changes
Parts:
- removed J5____JTAG: Conn_01x04, symbol Connector_Generic:Conn_01x04
- added C27: 10 μF, Capacitor_THT:C_Rect_L16.5mm_W4.7mm_P15.00mm_MKT, symbol Device:C
- added J5: Conn_01x06 JTAG, symbol Connector_Generic:Conn_01x06
- added R29: 100R, Resistor_SMD:R_0805_2012Metric_Pad1.20x1.40mm_HandSolder, symbol Device:R
- added SW1: SW_BIND_BT, symbol Switch:SW_Push
Connections:
- net GND: now also C27.2, SW1.2
- net MTCK: now reaches R27.1
- net MTCK: now also U2.16 (IO13)
- net at R27.2: now also J5.3 (Pin_3)
- net MTMS: now reaches R25.1
- net MTMS: now also U2.13 (IO14)
- net at R25.2: now also J5.1 (Pin_1)
- net MTDI: now reaches U2.14 (IO12)
- net MTDI: now also R26.1
- net MTDO: now reaches U2.23 (IO15)
- net MTDO: now also R28.1
- net at U2.28 (IO17): now also R29.2
- net at R26.2: now also J5.2 (Pin_2)
- net at R28.2: now also J5.4 (Pin_4)
- new net: C27.1, R29.1, SW1.1

Commit message: kicad update
Other:
- moved on the sheet: 998-MIC2779L-2YM5TR1, C15, C16, C17, C18, C19, C20, C25, C27, D6, D7, D8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
